File: board_def.kicad_sch (KiCad schematic)
At the start: 1 part

Commit message: more
Other:
- note added: "LENOVO SQUARE"
- note added: "MICRO_USB Female"
- moved on the sheet: D1

Commit message: latest
Parts:
- removed D1: LED, symbol Device:LED
Other:
- note added: "LED Diode"
Changed lines of the file:
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@@
+		)
+	)
+	(text "LED Diode"
+		(exclude_from_sim no)
+		(at 54.102 91.44 0)
+		(effects
+			(font
+				(size 1.27 1.27)
+			)
+			(justify left bottom)
 		)
 	)
@@
 		)
 	)
-	(symbol
-		(lib_id "Device:LED")
-		(at 60.96 91.44 0)
-		(unit 1)
-		(exclude_from_sim no)
-		(in_bom yes)
-		(on_board yes)
-		(dnp no)
-		(fields_autoplaced yes)
-		(property "Reference" "D1"
-			(at 59.3725 86.36 0)
-			(effects
-				(font
-					(size 1.27 1.27)
-				)
-			)
-		)
-		(property "Value" "LED"
-			(at 59.3725 88.9 0)
-			(effects
-				(font
-					(size 1.27 1.27)
-				)
-			)
-		)
-		(property "Footprint" ""
-			(at 60.96 91.44 0)
-			(effects
-				(font
-					(size 1.27 1.27)
-				)
-				(hide yes)
-			)
-		)
-		(property "Datasheet" "~"
-			(at 60.96 91.44 0)
-			(effects
-				(font
-					(size 1.27 1.27)
-				)
-				(hide yes)
-			)
-		)
-		(property "Description" ""
-			(at 60.96 91.44 0)
-			(effects
-				(font
-					(size 1.27 1.27)
-				)
-				(hide yes)
-			)
-		)
-		(pin "1"
-		)
-		(pin "2"
-		)
-		(instances
-			(project "dctester"
-				(path "/19eb1580-c65f-494d-88ac-d27fe4c49013/73d9d235-43d1-4b0c-a3da-7fb6c28a3a00"
-					(reference "D1")
-					(unit 1)
-				)
-			)
-		)
-	)
