File: dctester.kicad_pcb (KiCad board)
At the start: 2 copper layers, 50 x 65 mm, 15 parts, among them J1 Screw_Terminal_01x04, J2 USB_C_Receptacle_PowerOnly_6P, J3 Screw_Terminal_01x04, J5 USB_B_Micro, J6 DC5.5x2.1, J7 DC5.5x2.1

Commit message: Fix board and DRC
Parts:
- removed JP1, JP2: SolderJumper_3_Open, mypretties:SolderJumper-3_P4.0mm
- moved J2 7.52 mm to (131.5, 103.2)
- moved D2 5.59 mm to (107.5, 105.0)
- moved R1 3.54 mm to (115.0, 97.5)
- moved DJ2 1.64 mm to (131.8, 80.0)
- moved J5 1.46 mm to (130.4, 118.2)
- moved J7 1.44 mm to (121.5, 92.2)
Connections:
- D2 pad 1: GND -> outside
- DJ2 pad 1: GND -> outside
- DJ3 pad 1: GND -> outside
- DJ5 pad 1: GND -> outside
- DJ7 pad 1: GND -> outside
- DJ7 pad 2: GND -> outside
- J1 pad 2: Net-(J1-Pin_2) -> inside
- J1 pad 4: GND -> outside
- J2 pad A12: GND -> outside
- J2 pad B12: GND -> outside
- J2 pad S1: GND -> outside
- J3 pad 3: GND -> outside
- J3 pad 4: GND -> outside
- J5 pad 5: GND -> outside
- J5 pad 6: GND -> outside
- J6 pad 2: GND -> outside
- J6 pad 3: GND -> outside
Routing:
- net GND: track 308.4 -> 0.00 mm, vias 1 -> 0
- net outside: track 132.3 -> 376.1 mm
- net Net-(J1-Pin_2): track 32.0 -> 0.00 mm, vias 1 -> 0
- net inside: track 111.0 -> 136.6 mm, vias 1 -> 0
- net Net-(D2-A): track 15.6 -> 9.57 mm
- net /main/VDD: track 118.9 -> 120.1 mm, vias 1 -> 0
- added copper zone on F.Cu, net /main/VDD
- added copper zone on F.Cu, net inside
- added copper zone on B.Cu, net outside
Other:
- board size 50 x 65 mm -> 48.8 x 65 mm

Commit message: rev1.0
Other:
- board text added: "5.5x2.1"
- board text added: "5x5x2.5mm"
- board text added: "By LieBeDeMi Dec.2024"
- board text added: "DCTester rev1.0 DSN w/ KiCAD"
- board text added: "DJ3: 7.4x5.5mm"
- board text added: "DJ4: lenovo sqr"
- board text added: "DJ5: 5x5x2.5mm"
- board text added: "J1: 1/2: short or AMeter; 3/4: open or VMeter;"
- board text added: "J3: 1/2 VDD, 3/4 GND"
- board text added: "MyDigit.cn"
- board text added: "USB_C"
- board text added: "USB_micro"
- board text added: "hp_4.5x3mm"
Changed lines of the file:
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@@
 		(tags "Power Jack")
 		(property "Reference" "J7"
-			(at -11 -0.287852 0)
+			(at 2.792379 -3.608596 0)
 			(layer "F.SilkS")
 			(effects
@@
 		(at 131.8 80 -90)
 		(property "Reference" "DJ2"
-			(at 0 -2 -90)
+			(at -3.184419 10.46342 -90)
 			(unlocked yes)
 			(layer "F.SilkS")
@@
 		(at 97.5 120.74 90)
 		(property "Reference" "J3"
-			(at 11.25 -6.5 90)
+			(at 15.876791 3.601461 0)
 			(unlocked yes)
 			(layer "F.SilkS")
@@
 		(at 96.05 74 180)
 		(property "Reference" "DJ4"
-			(at 0.5 5 180)
+			(at 6.05 -3.5 0)
 			(unlocked yes)
 			(layer "F.SilkS")
@@
 		(tags "USB C Type-C receptacle power-only charging-only 6P 6C right angled")
 		(property "Reference" "J2"
-			(at 0 -5.1 90)
+			(at 2.660287 -5.691089 0)
 			(unlocked yes)
 			(layer "F.SilkS")
@@
 		(at 107.5 124.877306 180)
 		(property "Reference" "DJ7"
-			(at 0 9 180)
+			(at 5 14.877306 0)
 			(unlocked yes)
 			(layer "F.SilkS")
@@
 		(at 111.25 69.25)
 		(property "Reference" "DJ3"
-			(at -3 -2 0)
+			(at -3.75 5.75 0)
 			(unlocked yes)
 			(layer "F.SilkS")
@@
 		(tags "Power Jack")
 		(property "Reference" "J6"
-			(at -8.45 5.75 90)
+			(at -1.72172 8.4575 180)
 			(layer "F.SilkS")
 			(effects
@@
 		(at 124.75 61)
 		(property "Reference" "DJ5"
-			(at 0 9 0)
+			(at 7.75 1.5 0)
 			(unlocked yes)
 			(layer "F.SilkS")
@@
 		)
 	)
+	(gr_poly
+		(pts
+			(xy 100.167654 120.988398) (xy 100.600592 121.276714) (xy 100.600592 120.577561)
+		)
+		(stroke
+			(width 0.15)
+			(type solid)
+		)
+		(fill solid)
+		(layer "F.SilkS")
+	)
+	(gr_poly
+		(pts
+			(xy 114.39204 79.189387) (xy 114.680356 78.756449) (xy 113.981203 78.756449)
+		)
+		(stroke
+			(width 0.15)
+			(type solid)
+		)
+		(fill solid)
+		(layer "F.SilkS")
+	)
 	(gr_rect
 		(start 87 60)
@@
 		(layer "Edge.Cuts")
 	)
+	(gr_text "J1:\n1/2: short or AMeter;\n3/4: open or VMeter;"
+		(at 114.172817 90.753046 0)
+		(layer "B.SilkS")
+		(effects
+			(font
+				(size 1.5 1.5)
+				(thickness 0.2)
+				(bold yes)
+			)
+			(justify left bottom mirror)
+		)
+	)
+	(gr_text "USB_micro"
+		(at 134.209652 124.169122 0)
+		(layer "B.SilkS")
+		(effects
+			(font
+				(size 1 1)
+				(thickness 0.15)
+			)
+			(justify left bottom mirror)
+		)
+	)
+	(gr_text "5x5x2.5mm"
+		(at 111.836775 117.40604 0)
+		(layer "B.SilkS")
+		(effects
+			(font
+				(size 1 1)
+				(thickness 0.15)
+			)
+			(justify left bottom mirror)
+		)
+	)
+	(gr_text "5.5x2.1"
+		(at 133.458 95.874173 0)
+		(layer "B.SilkS")
+		(effects
+			(font
+				(size 1 1)
+				(thickness 0.15)
+			)
+			(justify left bottom mirror)
+		)
+	)
+	(gr_text "DJ4:\nlenovo sqr"
+		(at 99.384673 71.428704 0)
+		(layer "B.SilkS")
+		(effects
+			(font
+				(size 1 1)
+				(thickness 0.15)
+			)
+			(justify left bottom mirror)
+		)
+	)
+	(gr_text "DJ3: 7.4x5.5mm"
+		(at 117.113123 76.186217 0)
+		(layer "B.SilkS")
+		(effects
+			(font
+				(size 1 1)
+				(thickness 0.15)
+			)
+			(justify left bottom mirror)
+		)
+	)
+	(gr_text "By LieBeDeMi\nDec.2024"
+		(at 132.431836 105.911938 0)
+		(layer "B.SilkS" knockout)
+		(effects
+			(font
+				(size 2 2)
+				(thickness 0.2)
+			)
+			(justify left bottom mirror)
+		)
+	)
+	(gr_text "hp_4.5x3mm"
+		(at 134.794813 78.426905 0)
+		(layer "B.SilkS")
+		(effects
+			(font
+				(size 1 1)
+				(thickness 0.15)
+			)
+			(justify left bottom mirror)
+		)
+	)
+	(gr_text "MyDigit.cn"
+		(at 120 107.5 0)
+		(layer "B.SilkS")
+		(effects
+			(font
+				(size 1 1)
+				(thickness 0.15)
+			)
+			(justify left bottom mirror)
+		)
+	)
+	(gr_text "J3: 1/2 VDD, 3/4 GND"
+		(at 91.344412 95.195959 90)
+		(layer "B.SilkS")
+		(effects
+			(font
+				(size 1.5 1.6)
+				(thickness 0.2)
+			)
+			(justify left bottom mirror)
+		)
+	)
+	(gr_text "5.5x2.1"
+		(at 121.620612 123.080938 0)
+		(layer "B.SilkS")
+		(effects
+			(font
+				(size 1 1)
+				(thickness 0.15)
+			)
+			(justify left bottom mirror)
+		)
+	)
+	(gr_text "DJ5: 5x5x2.5mm"
+		(at 131.474765 69.475867 0)
+		(layer "B.SilkS")
+		(effects
+			(font
+				(size 1 1)
+				(thickness 0.15)
+			)
+			(justify left bottom mirror)
+		)
+	)
+	(gr_text "USB_C"
+		(at 133.678153 110 0)
+		(layer "B.SilkS")
+		(effects
+			(font
+				(size 1 1)
+				(thickness 0.15)
+			)
+			(justify left bottom mirror)
+		)
+	)
+	(gr_text "DCTester rev1.0\nDSN w/ KiCAD"
+		(at 113.699325 107.781878 0)
+		(layer "F.SilkS" knockout)
+		(effects
+			(font
+				(size 2 1)
+				(thickness 0.2)
+			)
+			(justify left bottom)
+		)
+	)
 	(segment
 		(start 110 105)
@@
 	)
 	(zone
-		(net 2)
-		(net_name "outside")
+		(net 3)
+		(net_name "inside")
 		(layer "F.Cu")
 		(name "$teardrop_padvia$")
 		(hatch full 0.1)
-		(priority 30002)
+		(priority 30003)
 		(attr
 			(teardrop
@@
 		(polygon
 			(pts
-				(xy 132.562531 117.744918) (xy 132.562531 118.744918) (xy 133.456928 118.969918) (xy 134.013531 118.244918)
-				(xy 133.456928 117.519918)
+				(xy 123.007442 81.190335) (xy 122.300335 81.897442) (xy 123.191694 82.313918) (xy 124.170707 81.960707)
+				(xy 124.249073 81.36)
 			)
 		)
@@
 		(name "$teardrop_padvia$")
 		(hatch full 0.1)
-		(priority 30003)
+		(priority 30000)
 		(attr
 			(teardrop
@@
 		(polygon
 			(pts
-				(xy 123.007442 81.190335) (xy 122.300335 81.897442) (xy 123.191694 82.313918) (xy 124.170707 81.960707)
-				(xy 124.249073 81.36)
+				(xy 105.357715 80.030608) (xy 104.650608 80.737715) (xy 105.34445 82.138663) (xy 106.620707 82.000707)
+				(xy 106.753963 80.71975)
 			)
 		)
@@
 	)
 	(zone
-		(net 3)
-		(net_name "inside")
+		(net 2)
+		(net_name "outside")
 		(layer "F.Cu")
 		(name "$teardrop_padvia$")
 		(hatch full 0.1)
-		(priority 30000)
+		(priority 30002)
 		(attr
 			(teardrop
@@
 		(polygon
 			(pts
-				(xy 105.357715 80.030608) (xy 104.650608 80.737715) (xy 105.34445 82.138663) (xy 106.620707 82.000707)
-				(xy 106.753963 80.71975)
+				(xy 132.562531 117.744918) (xy 132.562531 118.744918) (xy 133.456928 118.969918) (xy 134.013531 118.244918)
+				(xy 133.456928 117.519918)
+			)
+		)
+	)
+	(zone
+		(net 7)
+		(net_name "/main/VDD")
+		(layer "F.Cu")
+		(hatch edge 0.5)
+		(priority 3)
+		(connect_pads
+			(clearance 0.8)
+		)
+		(min_thickness 0.25)
+		(filled_areas_thickness no)
+		(fill yes
+			(thermal_gap 0.5)
+			(thermal_bridge_width 0.5)
+		)
+		(polygon
+			(pts
+				(xy 87.5 80) (xy 135 80) (xy 135 82.5) (xy 87.5 82.5)
+			)
+		)
+	)
+	(zone
+		(net 2)
+		(net_name "outside")
+		(layer "B.Cu")
+		(hatch edge 0.5)
+		(priority 2)
+		(connect_pads
+			(clearance 0.8)
+		)
+		(min_thickness 0.5)
+		(filled_areas_thickness no)
+		(fill yes
+			(thermal_gap 0.5)
+			(thermal_bridge_width 0.5)
+		)
+		(polygon
+			(pts
+				(xy 87.5 60) (xy 135 60) (xy 135 125) (xy 87.5 125)
 			)
 		)
@@
 			)
 		)
-	)
-	(zone
-		(net 2)
-		(net_name "outside")
-		(layer "B.Cu")
-		(hatch edge 0.5)
-		(priority 2)
-		(connect_pads
-			(clearance 0.8)
-		)
-		(min_thickness 0.5)
-		(filled_areas_thickness no)
-		(fill yes
-			(thermal_gap 0.5)
-			(thermal_bridge_width 0.5)
-		)
-		(polygon
-			(pts
-				(xy 87.5 60) (xy 135 60) (xy 135 125) (xy 87.5 125)
-			)
-		)
