File: main.kicad_sch (KiCad schematic)
At the start: 1 part

Commit message: latest
Parts:
- removed DJ1: ~, mypretties:lenovo_hp_dell_7.4x5mm_dc, symbol mylib:hp_dell_7.5x5.5mm_female
- added D2: LED, LED_THT:LED_D5.0mm, symbol Device:LED
- added DJ2: HP4.5x3, mypretties:hp_4.5x3.0mm_dc, symbol mylib:hp_4.5x3mm
- added DJ3: HP_DELL_LENOVO_7.4x5.5, mypretties:lenovo_hp_dell_7.4x5mm_dc, symbol mylib:hp_dell_7.5x5.5mm_female
- added DJ4: LENOVO_SQR, mypretties:lenovo_square_dc, symbol mylib:lenovo_square_dc
- added DJ5, DJ7: DC5.5x2.5, mypretties:general_5.5x2.5mm_dc, symbol mylib:general_dc5.5x2.5_female
- added J1, J3: Screw_Terminal_01x04, mypretties:screw762, symbol Connector:Screw_Terminal_01x04
- added J2: USB_C_Receptacle_PowerOnly_6P, mypretties:USB_C_Receptacle_GCT_USB4125-xx-x-0190_6P_TopMnt_Horizontal, symbol Connector:USB_C_Receptacle_PowerOnly_6P
- added J5: USB_B_Micro, mypretties:USB_Micro-B_flat_horizon, symbol Connector:USB_B_Micro
- added J6, J7: DC5.5x2.1, mypretties:BarrelJack_Horizontal, symbol Connector:Barrel_Jack_Switch
- added JP1, JP2: SolderJumper_3_Open, mypretties:SolderJumper-3_P4.0mm, symbol Jumper:SolderJumper_3_Open
- added R1: 2K, Resistor_THT:R_Axial_DIN0207_L6.3mm_D2.5mm_P10.16mm_Horizontal, symbol Device:R
Connections:
- new net: D2.2 (A), R1.1
- new net: J1.2 (Pin_2), JP1.2 (C)
- new net GND: D2.1 (K), DJ2.1 (shell), DJ3.1 (shell), DJ5.1 (shell), DJ7.1 (shell), DJ7.2 (outside), J1.4 (Pin_4), J2.A12 (GND), J2.B12 (GND), J2.S1 (SHIELD), J3.3 (Pin_3), J3.4 (Pin_4), J5.5 (GND), J5.6 (Shield), J6.2, J6.3, JP2.2 (C)
- new net VDD: DJ7.3 (inside), J1.1 (Pin_1), J1.3 (Pin_3), J2.A9 (VBUS), J2.B9 (VBUS), J3.1 (Pin_1), J3.2 (Pin_2), J5.1 (VBUS), J6.1, R1.2
- new net inside: DJ2.3 (inside), DJ3.3 (inside), DJ4.3 (inside), DJ5.3 (inside), J7.1, JP1.1 (A), JP2.3 (B)
- new net outside: DJ2.2 (outside), DJ3.2 (outside), DJ4.1 (shell), DJ4.2 (outside), DJ5.2 (outside), J7.2, J7.3, JP1.3 (B), JP2.1 (A)
- no-connect marks 0 -> 8
Other:
- note added: "J1: 1/2: short or A meter 3/4: open or V meter"
- note added: "J3: 1/2: VDD 3/4: GND"
- note added: "JP1/JP2: 12 inside = VDD 23 inside = GND"

Commit message: Fix board and DRC
Parts:
- removed JP1, JP2: SolderJumper_3_Open, mypretties:SolderJumper-3_P4.0mm, symbol Jumper:SolderJumper_3_Open
Connections:
- net outside is gone; now on net GND: DJ2.2 (outside), DJ3.2 (outside), DJ4.1 (shell), DJ4.2 (outside), DJ5.2 (outside), J7.2, J7.3
- net inside: now also J1.2 (Pin_2)
Other:
- note removed: "JP1/JP2: 12 inside = VDD 23 inside = GND"
